File: Whips-PCB/Whips-PCB.kicad_sch (KiCad schematic)
At the start: 33 parts, among them J1 12 VDC, J2 RS422 BUS, J3 SPEAKER 4OHM, J4 TO WHIP, J5 RS422 BUS, SW2 SW_DIP_x06, U2 MAX485ESA+T, U3 SN74AHCT125DR, U4 TSR_1-2450, U5 MAX98357AETE+T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

Commit message: Antenna 2026 initiated; new controller PCB
Parts:
- removed C4: 0.1uF, Capacitor_SMD:C_0402_1005Metric, symbol Device:C_Small
- removed C5: 10uF, Capacitor_SMD:C_0402_1005Metric, symbol Device:C_Small
- removed C6, C7: 220pF, Capacitor_SMD:C_0402_1005Metric, symbol Device:C_Small
- removed D3, D4: LED, Joels KiCad Footprint Library:Everlight 99-218GLM2C-L7277SGU-TR8-T0-ES side view LED, symbol Device:LED
- removed H1: DNP (LOGO), Joels KiCad Footprint Library:Turtle-Art-2024, symbol Mechanical:MountingHole
- removed J1: 12 VDC, TerminalBlock_Phoenix:TerminalBlock_Phoenix_MKDS-1,5-2_1x02_P5.00mm_Horizontal, symbol Connector_Generic:Conn_01x02
- removed J2, J5: RS422 BUS, TerminalBlock_Phoenix:TerminalBlock_Phoenix_MKDS-1,5-2_1x02_P5.00mm_Horizontal, symbol Connector_Generic:Conn_01x02
- removed J3: SPEAKER 4OHM, TerminalBlock_Phoenix:TerminalBlock_Phoenix_MKDS-1,5-2_1x02_P5.00mm_Horizontal, symbol Connector_Generic:Conn_01x02
- removed J4: TO WHIP, TerminalBlock_Phoenix:TerminalBlock_Phoenix_MKDS-1,5-3_1x03_P5.00mm_Horizontal, symbol Connector_Generic:Conn_01x03
- removed R10, R11: 470, Resistor_SMD:R_0402_1005Metric, symbol Device:R_US
- removed R7: 1M, Resistor_SMD:R_0402_1005Metric, symbol Device:R_US
- removed R8: 100K, Resistor_SMD:R_0402_1005Metric, symbol Device:R_US
- removed SW2: SW_DIP_x06, Button_Switch_THT:SW_DIP_SPSTx06_Slide_6.7x16.8mm_W7.62mm_P2.54mm_LowProfile, symbol Switch:SW_DIP_x06
- removed U5: MAX98357AETE+T, Joels KiCad Footprint Library:MAX98357AETE+T, symbol Joels KiCad Symbol Library:MAX98357AETE+T
- added J2: Conn_01x05_Socket, Joels KiCad Footprint Library:Dorabo_DB103-5.0-5P-GN-S, symbol Connector:Conn_01x05_Socket
- added SW1: DSWB06LHGET, Joels KiCad Footprint Library:DongGuan_DSWB06LHGET_6_PIN_DIP, symbol Joels KiCad Symbol Library:DongGuan_DSWB06LHGET_DIP_6_SWITCH
Connections:
- net 12VDC: now also J2.1 (Pin_1)
- net GND: now also J2.5 (Pin_5), SW1.10, SW1.11, SW1.12, SW1.8, SW1.9
- net NEO: now also J2.2 (Pin_2)
- net at U6.4 (2_OUT2): now also SW1.2
- net at U6.5 (3_LRCLK2): now also SW1.3
- net at U6.6 (4_BCLK2): now also SW1.4
- net at U6.7 (5_IN2): now also SW1.5
- net at U6.8 (6_OUT1D): now also SW1.6
- net at R5.1: now also SW1.1
- net A renamed RS422-A
- net RS422-A: now also J2.3 (Pin_3), SW1.7
- net B renamed RS422-B
- net RS422-B: now also J2.4 (Pin_4)
- net BCLK: no longer names the net of U6.43 (21_A7_RX5_BCLK1)
- net DAT: no longer names the net of U6.9 (7_RX2_OUT1A)
- net LRCLK: no longer names the net of U6.42 (20_A6_TX5_LRCLK1)
- no-connect marks 38 -> 41
Other:
- note removed: "side lights for turtle logo"
